File: PCB/kicad/Peghammer_wirelessB/Peghammer_wirelessB.kicad_sch (KiCad schematic)
At the start: 30 parts, among them P1 ピンヘッダ_01x04_オス, P2 ピンヘッダ_01x04_オス, P3 ピンヘッダ_01x04_オス, P4 ピンヘッダ_01x04_オス, P5 ピンヘッダ_01x04_オス

Commit message: Add files via upload
Connections:
- net GND: now also P1.3 (Pin_3), P2.3 (Pin_3), P5.4 (Pin_4), S1.3 (Pin_3), S2.3 (Pin_3), SW18.1 (com)
- no-connect marks 9 -> 7
